File: Punkys-new-brew_control.kicad_pcb (KiCad board)
At the start: 2 copper layers, 40.1 x 110 mm, 21 parts, among them J10 VCA-CV, J12 1x10_control, J14 L_1x12_control, J15 R_1x12_control, J2 CV1-In, J3 CV2-In, J4 Gate-In, J5 Audio-Out, J6 Ext-Audio, J7 ENV1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

Commit message: fixed some values to better suit my liking. re-routed the invert to env2 instead, it works better me finks.
Parts:
- RV1: value 500k -> 1M
- RV7: value 1M -> 500k
Routing:
- net GND: vias 7 -> 6
Changed lines of the file:
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@@
     (title "Punky's New Brew")
     (date "2023-10-20")
-    (rev "001")
+    (rev "003")
     (company "Scruffy Cat Studios @2023")
   )
@@
         (effects (font (size 1 1) (thickness 0.15)))
     )
-    (fp_text value "1M" (at 0 10.11 90) (layer "F.Fab")
+    (fp_text value "500k" (at 0 10.11 90) (layer "F.Fab")
         (effects (font (size 1 1) (thickness 0.15)))
     )
@@
         (effects (font (size 1 1) (thickness 0.15)))
     )
-    (fp_text value "500k" (at 0 10.11 90) (layer "F.Fab")
+    (fp_text value "1M" (at 0 10.11 90) (layer "F.Fab")
         (effects (font (size 1 1) (thickness 0.15)))
     )
@@
   (via (at 150.96 64.38) (size 0.8) (drill 0.4) (layers "F.Cu" "B.Cu") (free) (net 2))
   (via (at 140.33 53.32) (size 0.8) (drill 0.4) (layers "F.Cu" "B.Cu") (free) (net 2))
-  (via (at 121.65 135.66) (size 0.6) (drill 0.3) (layers "F.Cu" "B.Cu") (free) (net 2))
   (via (at 157.03 49.96) (size 0.8) (drill 0.4) (layers "F.Cu" "B.Cu") (free) (net 2))
   (via (at 150.55 85.07) (size 0.8) (drill 0.4) (layers "F.Cu" "B.Cu") (free) (net 2))
